File: ESP32_DevKit_C_v4-AZDelivery_Breadboard_Adapter.kicad_pcb (KiCad board)
At the start: 4 copper layers, 133 x 29 mm, 9 parts, among them J1 Conn_01x19_Female, J2 Conn_01x19_Female, J3 Conn_01x18_Male, J4 Conn_01x18_Male, J5 Conn_01x04_Female

Commit message: v2
Other:
- board text added: "+"
- board text added: "-"
Changed lines of the file:
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@@
     )
     (fp_line (start -0.994955 -1.084158) (end 3.511561 -1.08179) (layer "F.SilkS") (width 0.12))
-    (fp_arc (start 3.511561 -1.08179) (mid 1.256419 2.5) (end -0.994955 -1.084158) (layer "F.SilkS") (width 0.12))
+    (fp_arc (start 3.511561 -1.08179) (mid 1.25642 2.499999) (end -0.994955 -1.084158) (layer "F.SilkS") (width 0.12))
     (fp_line (start -1.95 3.25) (end 4.5 3.25) (layer "F.CrtYd") (width 0.05))
     (fp_line (start 4.5 3.25) (end 4.5 -3.25) (layer "F.CrtYd") (width 0.05))
@@
     (effects (font (size 1 1) (thickness 0.15)))
   )
+  (gr_text "+" (at 125.19 80.22) (layer "F.SilkS")
+    (effects (font (size 1 1) (thickness 0.15)))
+  )
   (gr_text "LED\nGPIO 2" (at 128.3 76.2) (layer "F.SilkS")
     (effects (font (size 1 1) (thickness 0.15)))
@@
     (effects (font (size 0.6 0.6) (thickness 0.15)))
   )
+  (gr_text "-" (at 131.51 80.2) (layer "F.SilkS")
+    (effects (font (size 1 1) (thickness 0.15)))
+  )
   (gr_text "13" (at 172.72 65.786 270) (layer "F.SilkS")
